File: motordriver.sch (EAGLE design)
At the start: 0 parts

Commit message: Changed schematic
Suck it.
Parts:
- added Q1: MOSFET, motordriverslib:MOSFET
Changed lines of the file:
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@@
 <?xml version="1.0" encoding="utf-8"?>
 <!DOCTYPE eagle SYSTEM "eagle.dtd">
-<eagle version="7.1.0">
+<eagle version="7.2.0">
 <drawing>
 <settings>
@@
 <layer number="48" name="Document" color="7" fill="1" visible="no" active="no"/>
 <layer number="49" name="Reference" color="7" fill="1" visible="no" active="no"/>
+<layer number="50" name="dxf" color="7" fill="1" visible="no" active="no"/>
 <layer number="51" name="tDocu" color="7" fill="1" visible="no" active="no"/>
 <layer number="52" name="bDocu" color="7" fill="1" visible="no" active="no"/>
+<layer number="53" name="tGND_GNDA" color="7" fill="9" visible="no" active="no"/>
+<layer number="54" name="bGND_GNDA" color="1" fill="9" visible="no" active="no"/>
+<layer number="56" name="wert" color="7" fill="1" visible="no" active="no"/>
 <layer number="90" name="Modules" color="5" fill="1" visible="yes" active="yes"/>
 <layer number="91" name="Nets" color="2" fill="1" visible="yes" active="yes"/>
@@
 <layer number="97" name="Info" color="7" fill="1" visible="yes" active="yes"/>
 <layer number="98" name="Guide" color="6" fill="1" visible="yes" active="yes"/>
+<layer number="100" name="Muster" color="7" fill="1" visible="no" active="no"/>
+<layer number="101" name="Patch_Top" color="12" fill="4" visible="no" active="yes"/>
+<layer number="102" name="Vscore" color="7" fill="1" visible="no" active="yes"/>
+<layer number="103" name="tMap" color="7" fill="1" visible="no" active="yes"/>
+<layer number="104" name="Name" color="16" fill="1" visible="no" active="yes"/>
+<layer number="105" name="tPlate" color="7" fill="1" visible="no" active="yes"/>
+<layer number="106" name="bPlate" color="7" fill="1" visible="no" active="yes"/>
+<layer number="107" name="Crop" color="7" fill="1" visible="no" active="yes"/>
+<layer number="108" name="tplace-old" color="10" fill="1" visible="yes" active="yes"/>
+<layer number="109" name="ref-old" color="11" fill="1" visible="yes" active="yes"/>
+<layer number="116" name="Patch_BOT" color="9" fill="4" visible="no" active="yes"/>
+<layer number="121" name="_tsilk" color="7" fill="1" visible="no" active="yes"/>
+<layer number="122" name="_bsilk" color="7" fill="1" visible="no" active="yes"/>
+<layer number="125" name="_tNames" color="7" fill="1" visible="no" active="yes"/>
+<layer number="144" name="Drill_legend" color="7" fill="1" visible="no" active="yes"/>
+<layer number="151" name="HeatSink" color="7" fill="1" visible="no" active="yes"/>
+<layer number="199" name="Contour" color="7" fill="1" visible="yes" active="yes"/>
+<layer number="200" name="200bmp" color="1" fill="10" visible="no" active="yes"/>
+<layer number="201" name="201bmp" color="2" fill="10" visible="no" active="yes"/>
+<layer number="202" name="202bmp" color="3" fill="10" visible="no" active="yes"/>
+<layer number="203" name="203bmp" color="4" fill="10" visible="no" active="yes"/>
+<layer number="204" name="204bmp" color="5" fill="10" visible="no" active="yes"/>
+<layer number="205" name="205bmp" color="6" fill="10" visible="no" active="yes"/>
+<layer number="206" name="206bmp" color="7" fill="10" visible="no" active="yes"/>
+<layer number="207" name="207bmp" color="8" fill="10" visible="no" active="yes"/>
+<layer number="208" name="208bmp" color="9" fill="10" visible="no" active="yes"/>
+<layer number="209" name="209bmp" color="7" fill="1" visible="no" active="yes"/>
+<layer number="210" name="210bmp" color="7" fill="1" visible="no" active="yes"/>
+<layer number="211" name="211bmp" color="7" fill="1" visible="no" active="yes"/>
+<layer number="212" name="212bmp" color="7" fill="1" visible="no" active="yes"/>
+<layer number="213" name="213bmp" color="7" fill="1" visible="no" active="yes"/>
+<layer number="214" name="214bmp" color="7" fill="1" visible="no" active="yes"/>
+<layer number="215" name="215bmp" color="7" fill="1" visible="no" active="yes"/>
+<layer number="216" name="216bmp" color="7" fill="1" visible="no" active="yes"/>
+<layer number="217" name="217bmp" color="18" fill="1" visible="no" active="no"/>
+<layer number="218" name="218bmp" color="19" fill="1" visible="no" active="no"/>
+<layer number="219" name="219bmp" color="20" fill="1" visible="no" active="no"/>
+<layer number="220" name="220bmp" color="21" fill="1" visible="no" active="no"/>
+<layer number="221" name="221bmp" color="22" fill="1" visible="no" active="no"/>
+<layer number="222" name="222bmp" color="23" fill="1" visible="no" active="no"/>
+<layer number="223" name="223bmp" color="24" fill="1" visible="no" active="no"/>
+<layer number="224" name="224bmp" color="25" fill="1" visible="no" active="no"/>
+<layer number="250" name="Descript" color="3" fill="1" visible="no" active="no"/>
+<layer number="251" name="SMDround" color="12" fill="11" visible="no" active="no"/>
+<layer number="254" name="cooling" color="7" fill="1" visible="no" active="yes"/>
 </layers>
 <schematic xreflabel="%F%N/%S.%C%R" xrefpart="/%S.%C%R">
@@
 </classes>
 <parts>
+<part name="Q1" library="motordriverslib" deviceset="MOSFET" device=""/>
 </parts>
 <sheets>
@@
 </plain>
 <instances>
+<instance part="Q1" gate="G$1" x="12.7" y="71.12"/>
 </instances>
 <busses>

Commit message: Testing the save function
Dicks
Parts:
- added U1: TL084_PDIP, motordriverslib:TL084_PDIP
Changed lines of the file:
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@@
 <parts>
 <part name="Q1" library="motordriverslib" deviceset="MOSFET" device=""/>
+<part name="U1" library="motordriverslib" deviceset="TL084_PDIP" device=""/>
 </parts>
 <sheets>
@@
 <instances>
 <instance part="Q1" gate="G$1" x="12.7" y="71.12"/>
+<instance part="U1" gate="G$1" x="-10.16" y="71.12"/>
 </instances>
 <busses>

Commit message: Initial schat
Parts:
- added C1: CAP_1U, motordriverslib:CAP_1U
- added J1: CONNECTOR_MOTORS, motordriverslib:CONNECTOR_MOTORS
- added Q2, Q3, Q4: MOSFET, motordriverslib:MOSFET
- added U2: TL084_PDIP, motordriverslib:TL084_PDIP
- added U3: 7812_TO220, motordriverslib:7812_TO220
- added U5: IR2111_PDIP, motordriverslib:IR2111_PDIP
- U1: value TL084_PDIP -> 74XX139_PDIP; device motordriverslib:TL084_PDIP -> motordriverslib:74XX139_PDIP
Connections:
- new net GND: U3.GND
- new net N$1: U1.P$11, U2.4-
- new net N$10: U2.OUT1, U5.P$2
- new net N$11: C1.2, U3.OUT, U5.P$1
- new net N$12: C1.1, U5.P$3
- new net N$2: U2.3+, U2.4+
- new net N$3: U2.1+, U2.2+
- new net N$4: U1.P$5, U2.1-
- new net N$5: U1.P$7, U2.2-
- new net N$6: U1.P$9, U2.3-
- new net N$7: U2.OUT3
- new net N$8: U2.OUT2
- new net N$9: U2.OUT4
- new net VCC: U3.IN
Other:
- moved on the sheet: Q1
Changed lines of the file:
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@@
 </classes>
 <parts>
+<part name="U1" library="motordriverslib" deviceset="74XX139_PDIP" device=""/>
+<part name="U2" library="motordriverslib" deviceset="TL084_PDIP" device=""/>
+<part name="U3" library="motordriverslib" deviceset="7812_TO220" device=""/>
+<part name="J1" library="motordriverslib" deviceset="CONNECTOR_MOTORS" device=""/>
+<part name="U5" library="motordriverslib" deviceset="IR2111_PDIP" device=""/>
 <part name="Q1" library="motordriverslib" deviceset="MOSFET" device=""/>
-<part name="U1" library="motordriverslib" deviceset="TL084_PDIP" device=""/>
+<part name="Q2" library="motordriverslib" deviceset="MOSFET" device=""/>
+<part name="Q3" library="motordriverslib" deviceset="MOSFET" device=""/>
+<part name="Q4" library="motordriverslib" deviceset="MOSFET" device=""/>
+<part name="GND1" library="supply1" deviceset="GND" device=""/>
+<part name="P+1" library="supply1" deviceset="VCC" device=""/>
+<part name="C1" library="motordriverslib" deviceset="CAP_1U" device=""/>
 </parts>
 <sheets>
@@
 </plain>
 <instances>
-<instance part="Q1" gate="G$1" x="12.7" y="71.12"/>
-<instance part="U1" gate="G$1" x="-10.16" y="71.12"/>
+<instance part="U1" gate="G$1" x="-185.42" y="-5.08"/>
+<instance part="U2" gate="G$1" x="-182.88" y="33.02"/>
+<instance part="U3" gate="G$1" x="-106.68" y="71.12"/>
+<instance part="J1" gate="G$1" x="-218.44" y="101.6"/>
+<instance part="U5" gate="G$1" x="-63.5" y="48.26"/>
+<instance part="Q1" gate="G$1" x="-218.44" y="78.74"/>
+<instance part="Q2" gate="G$1" x="-198.12" y="86.36"/>
+<instance part="Q3" gate="G$1" x="-180.34" y="76.2"/>
+<instance part="Q4" gate="G$1" x="-157.48" y="81.28"/>
+<instance part="GND1" gate="1" x="-106.68" y="63.5"/>
+<instance part="P+1" gate="VCC" x="-121.92" y="99.06"/>
+<instance part="C1" gate="G$1" x="-81.28" y="53.34" rot="R180"/>
 </instances>
 <busses>
 </busses>
 <nets>
+<net name="N$1" class="0">
+<segment>
+<pinref part="U2" gate="G$1" pin="4-"/>
+<wire x1="-175.26" y1="53.34" x2="-157.48" y2="53.34" width="0.1524" layer="91"/>
+<wire x1="-157.48" y1="53.34" x2="-157.48" y2="-10.16" width="0.1524" layer="91"/>
+<pinref part="U1" gate="G$1" pin="P$11"/>
+<wire x1="-157.48" y1="-10.16" x2="-175.26" y2="-10.16" width="0.1524" layer="91"/>
+</segment>
+</net>
+<net name="N$2" class="0">
+<segment>
+<pinref part="U2" gate="G$1" pin="4+"/>
+<wire x1="-175.26" y1="48.26" x2="-170.18" y2="48.26" width="0.1524" layer="91"/>
+<wire x1="-170.18" y1="48.26" x2="-170.18" y2="38.1" width="0.1524" layer="91"/>
+<pinref part="U2" gate="G$1" pin="3+"/>
+<wire x1="-170.18" y1="38.1" x2="-175.26" y2="38.1" width="0.1524" layer="91"/>
+</segment>
+</net>
+<net name="N$3" class="0">
+<segment>
+<pinref part="U2" gate="G$1" pin="1+"/>
+<wire x1="-190.5" y1="48.26" x2="-195.58" y2="48.26" width="0.1524" layer="91"/>
+<wire x1="-195.58" y1="48.26" x2="-195.58" y2="38.1" width="0.1524" layer="91"/>
+<pinref part="U2" gate="G$1" pin="2+"/>
+<wire x1="-195.58" y1="38.1" x2="-190.5" y2="38.1" width="0.1524" layer="91"/>
+</segment>
+</net>
+<net name="N$4" class="0">
+<segment>
+<pinref part="U2" gate="G$1" pin="1-"/>
+<wire x1="-190.5" y1="53.34" x2="-205.74" y2="53.34" width="0.1524" layer="91"/>
+<wire x1="-205.74" y1="53.34" x2="-205.74" y2="-5.08" width="0.1524" layer="91"/>
+<pinref part="U1" gate="G$1" pin="P$5"/>
+<wire x1="-205.74" y1="-5.08" x2="-190.5" y2="-5.08" width="0.1524" layer="91"/>
+</segment>
+</net>
+<net name="N$5" class="0">
+<segment>
+<pinref part="U1" gate="G$1" pin="P$7"/>
+<wire x1="-190.5" y1="-15.24" x2="-200.66" y2="-15.24" width="0.1524" layer="91"/>
+<wire x1="-200.66" y1="-15.24" x2="-200.66" y2="33.02" width="0.1524" layer="91"/>
+<pinref part="U2" gate="G$1" pin="2-"/>
+<wire x1="-200.66" y1="33.02" x2="-190.5" y2="33.02" width="0.1524" layer="91"/>
+</segment>
+</net>
+<net name="N$6" class="0">
+<segment>
+<pinref part="U2" gate="G$1" pin="3-"/>
+<wire x1="-175.26" y1="33.02" x2="-167.64" y2="33.02" width="0.1524" layer="91"/>
+<wire x1="-167.64" y1="33.02" x2="-167.64" y2="-20.32" width="0.1524" layer="91"/>
+<pinref part="U1" gate="G$1" pin="P$9"/>
+<wire x1="-167.64" y1="-20.32" x2="-175.26" y2="-20.32" width="0.1524" layer="91"/>
+</segment>
+</net>
+<net name="N$7" class="0">
+<segment>
+<pinref part="U2" gate="G$1" pin="OUT3"/>
+<wire x1="-175.26" y1="27.94" x2="-139.7" y2="27.94" width="0.1524" layer="91"/>
+</segment>
+</net>
+<net name="N$8" class="0">
+<segment>
+<pinref part="U2" gate="G$1" pin="OUT2"/>
+<wire x1="-190.5" y1="27.94" x2="-226.06" y2="27.94" width="0.1524" layer="91"/>
+</segment>
+</net>
+<net name="N$9" class="0">
+<segment>
+<pinref part="U2" gate="G$1" pin="OUT4"/>
+<wire x1="-175.26" y1="58.42" x2="-139.7" y2="58.42" width="0.1524" layer="91"/>
+</segment>
+</net>
+<net name="VCC" class="0">
+<segment>
+<pinref part="U3" gate="G$1" pin="IN"/>
+<wire x1="-114.3" y1="73.66" x2="-121.92" y2="73.66" width="0.1524" layer="91"/>
+<wire x1="-121.92" y1="73.66" x2="-121.92" y2="96.52" width="0.1524" layer="91"/>
+<pinref part="P+1" gate="VCC" pin="VCC"/>
+</segment>
+</net>
+<net name="GND" class="0">
+<segment>
+<pinref part="U3" gate="G$1" pin="GND"/>
+<pinref part="GND1" gate="1" pin="GND"/>
+</segment>
+</net>
+<net name="N$11" class="0">
+<segment>
+<pinref part="U3" gate="G$1" pin="OUT"/>
+<wire x1="-99.06" y1="73.66" x2="-81.28" y2="73.66" width="0.1524" layer="91"/>
+<wire x1="-81.28" y1="73.66" x2="-81.28" y2="55.88" width="0.1524" layer="91"/>
+<pinref part="U5" gate="G$1" pin="P$1"/>
+<wire x1="-81.28" y1="55.88" x2="-71.12" y2="55.88" width="0.1524" layer="91"/>
+<pinref part="C1" gate="G$1" pin="2"/>
+<junction x="-81.28" y="55.88"/>
+</segment>
+</net>
+<net name="N$12" class="0">
+<segment>
+<pinref part="C1" gate="G$1" pin="1"/>
+<wire x1="-81.28" y1="48.26" x2="-81.28" y2="45.72" width="0.1524" layer="91"/>
+<pinref part="U5" gate="G$1" pin="P$3"/>
+<wire x1="-81.28" y1="45.72" x2="-71.12" y2="45.72" width="0.1524" layer="91"/>
+</segment>
+</net>
+<net name="N$10" class="0">
+<segment>
+<pinref part="U2" gate="G$1" pin="OUT1"/>
+<wire x1="-190.5" y1="58.42" x2="-200.66" y2="58.42" width="0.1524" layer="91"/>
+<wire x1="-200.66" y1="58.42" x2="-200.66" y2="66.04" width="0.1524" layer="91"/>
+<wire x1="-200.66" y1="66.04" x2="-116.84" y2="66.04" width="0.1524" layer="91"/>
+<wire x1="-116.84" y1="66.04" x2="-116.84" y2="58.42" width="0.1524" layer="91"/>
+<wire x1="-116.84" y1="58.42" x2="-76.2" y2="58.42" width="0.1524" layer="91"/>
+<wire x1="-76.2" y1="58.42" x2="-76.2" y2="50.8" width="0.1524" layer="91"/>
+<pinref part="U5" gate="G$1" pin="P$2"/>
+<wire x1="-76.2" y1="50.8" x2="-71.12" y2="50.8" width="0.1524" layer="91"/>
+</segment>
+</net>
 </nets>
 </sheet>

Commit message: Basic completed driver Schematic
Need the Dode, 5v LDO, and miscellaneous connector footprints
Parts:
- added C10, C14, C16, C2, C20, C22, C4, C8: CAP_2200U_63V, motordriverslib:CAP_2200U_63V
- added C11, C12, C13, C15, C17, C18, C19, C21, C23, C24, C3, C5, C6, C7, C9: CAP_1U, motordriverslib:CAP_1U
- added D1, D2, D3, D4, D5, D6, D7, D8: 1N4004, diode:1N4004
- added J2, J3, J4: CONNECTOR_MOTORS, motordriverslib:CONNECTOR_MOTORS
- added Q10, Q11, Q12, Q13, Q14, Q15, Q16, Q5, Q6, Q7, Q8, Q9: MOSFET, motordriverslib:MOSFET
- added R1, R10, R11, R12, R13, R14, R15, R16, R2, R3, R4, R5, R6, R7, R8, R9: RES_SMT, motordriverslib:RES_SMT
- added U10, U11, U4, U6, U7, U8, U9: IR2111_PDIP, motordriverslib:IR2111_PDIP
Connections:
- removed net N$11: C1.2, U3.OUT, U5.P$1
- removed net N$12: C1.1, U5.P$3
- removed net N$9: U2.OUT4
- new net N$13: C2.+, D1.C, U5.P$8
- new net N$14: Q1.G, R4.2
- new net N$15: C2.-, U5.P$6
- new net N$16: R1.1, U5.P$7
- new net N$17: Q4.G, R1.2
- new net N$18: J1.+, Q3.D, Q4.S
- new net N$19: R4.1, U5.P$4
- new net N$20: R3.1, U4.P$4
- new net N$21: J1.-, Q1.D, Q2.S
- new net N$22: Q3.G, R3.2
- new net N$24: Q2.G, R2.2
- new net N$25: C4.+, D2.C, U4.P$8
- new net N$26: C4.-, U4.P$6
- new net N$27: R2.1, U4.P$7
- new net N$30: C8.+, D3.C, U6.P$8
- new net N$31: C8.-, U6.P$6
- new net N$32: R5.1, U6.P$7
- new net N$33: Q8.G, R5.2
- new net N$34: J2.+, Q7.D, Q8.S
- new net N$35: R8.1, U6.P$4
- new net N$36: Q5.G, R8.2
- new net N$37: J2.-, Q5.D, Q6.S
- new net N$38: C10.+, D4.C, U7.P$8
- new net N$39: C10.-, U7.P$6
- new net N$40: R6.1, U7.P$7
- new net N$41: R7.1, U7.P$4
- new net N$42: Q7.G, R7.2
- new net N$43: Q6.G, R6.2
- new net N$44: U11.P$2, U2.OUT1, U9.P$2
- new net N$47: C14.+, D5.C, U8.P$8
- new net N$48: C14.-, U8.P$6
- new net N$49: R9.1, U8.P$7
- new net N$50: Q12.G, R9.2
- new net N$51: J3.+, Q11.D, Q12.S
- new net N$52: R12.1, U8.P$4
- new net N$53: Q9.G, R12.2
- new net N$54: J3.-, Q10.S, Q9.D
- new net N$55: C16.+, D6.C, U9.P$8
- new net N$56: C16.-, U9.P$6
- new net N$57: R10.1, U9.P$7
- new net N$58: R11.1, U9.P$4
- new net N$59: Q11.G, R11.2
- new net N$60: Q10.G, R10.2
- new net N$63: U10.P$2, U2.OUT2, U8.P$2
- new net N$64: C20.+, D7.C, U10.P$8
- new net N$65: C20.-, U10.P$6
- new net N$66: R13.1, U10.P$7
- new net N$67: Q16.G, R13.2
- new net N$68: J4.+, Q15.D, Q16.S
- new net N$69: R16.1, U10.P$4
- new net N$70: Q13.G, R16.2
- new net N$71: J4.-, Q13.D, Q14.S
- new net N$72: C22.+, D8.C, U11.P$8
- new net N$73: C22.-, U11.P$6
- new net N$74: R14.1, U11.P$7
- new net N$75: R15.1, U11.P$4
- new net N$76: Q15.G, R15.2
- new net N$77: Q14.G, R14.2
- net GND: now also C1.1, C11.1, C12.2, C13.1, C15.1, C17.1, C18.2, C19.1, C21.1, C23.1, C24.2, C3.1, C5.1, C6.2, C7.1, C9.1, Q1.S, Q11.S, Q13.S, Q15.S, Q3.S, Q5.S, Q7.S, Q9.S, U10.P$3, U11.P$3, U4.P$3, U5.P$3, U6.P$3, U7.P$3, U8.P$3, U9.P$3
- net N$10: now also U2.OUT4, U6.P$2; no longer U2.OUT1
- net N$7: now also U4.P$2, U7.P$2
- net N$8: now also C1.2, C13.2, C15.2, C19.2, C21.2, C3.2, C7.2, C9.2, D1.A, D2.A, D3.A, D4.A, D5.A, D6.A, D7.A, D8.A, U10.P$1, U11.P$1, U3.OUT, U4.P$1, U5.P$1, U6.P$1, U7.P$1, U8.P$1, U9.P$1; no longer U2.OUT2
- net VCC: now also C11.2, C12.1, C17.2, C18.1, C23.2, C24.1, C5.2, C6.1, Q10.D, Q12.D, Q14.D, Q16.D, Q2.D, Q4.D, Q6.D, Q8.D
Other:
- moved on the sheet: J1, Q1, Q2, Q3, Q4, U3

Commit message: Changed schematic
Connections:
- removed net N$8: C1.2, C13.2, C15.2, C19.2, C21.2, C3.2, C7.2, C9.2, D1.A, D2.A, D3.A, D4.A, D5.A, D6.A, D7.A, D8.A, U10.P$1, U11.P$1, U3.OUT, U4.P$1, U5.P$1, U6.P$1, U7.P$1, U8.P$1, U9.P$1
- new net V_IN: U3.IN
- net VCC: now also C1.2, C13.2, C15.2, C19.2, C21.2, C3.2, C7.2, C9.2, D1.A, D2.A, D3.A, D4.A, D5.A, D6.A, D7.A, D8.A, U10.P$1, U11.P$1, U3.OUT, U4.P$1, U5.P$1, U6.P$1, U7.P$1, U8.P$1, U9.P$1; no longer U3.IN
Other:
- note added: "add power switch add bulk power decoupling change caps and diodes move motor decouplers add encoder connectors add fan LDO and header pins (12v)"

Commit message: Schematic changes
Added power switch, power decoups, moter decoups, fan connections
Parts:
- removed C17, C18: CAP_1U, motordriverslib:CAP_1U
- added J5, J6: HEADER_1X3, motordriverslib:HEADER_1X3
- added S1: ROCKER_THRU, motordriverslib:ROCKER_THRU
- added U$1: 7805_TO220, motordriverslib:7805_TO220
- C23, C24: value CAP_1U -> CAP_2200U_63V; device motordriverslib:CAP_1U -> motordriverslib:CAP_2200U_63V
Connections:
- new net N$11: U$1.OUT, U1.P$16, U2.VCC
- new net N$12: J5.2
- new net N$23: J5.3
- new net N$28: J6.3
- new net N$29: J6.2
- new net N$8: U$1.IN
- net GND: now also C23.-, C24.-, J5.1, J6.1, U$1.GND, U1.P$8, U2.GND; no longer C11.1, C12.2, C17.1, C18.2, C23.1, C24.2, C5.1, C6.2
- net N$18: now also C11.1
- net N$21: now also C11.2
- net N$34: now also C12.1
- net N$37: now also C12.2
- net N$51: now also C5.1
- net N$54: now also C5.2
- net N$68: now also C6.1
- net N$71: now also C6.2
- net VCC: now also C23.+, C24.+, S1.+; no longer C11.2, C12.1, C17.2, C18.1, C23.2, C24.1, C5.2, C6.1
- net V_IN: now also S1.-
Other:
- note added: "5 V LDO"
- note added: "<done>"
- note added: "done"
- note added: "dunzo"
- moved on the sheet: C11, C12, C5, C6

Commit message: FIXED STUFF
Connections:
- net VCC renamed VCC_12V
Changed lines of the file:
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@@
 <?xml version="1.0" encoding="utf-8"?>
 <!DOCTYPE eagle SYSTEM "eagle.dtd">
-<eagle version="7.2.0">
+<eagle version="7.1.0">
 <drawing>
 <settings>
@@
 </segment>
 </net>
-<net name="VCC" class="0">
+<net name="VCC_12V" class="0">
 <segment>
 <pinref part="P+5" gate="VCC" pin="VCC"/>
@@
 <wire x1="-175.26" y1="83.82" x2="-165.1" y2="83.82" width="0.1524" layer="91"/>
 <wire x1="-165.1" y1="83.82" x2="-86.36" y2="83.82" width="0.1524" layer="91"/>
-<wire x1="-86.36" y1="83.82" x2="116.84" y2="83.82" width="0.1524" layer="91"/>
-<pinref part="U4" gate="G$1" pin="P$1"/>
-<wire x1="116.84" y1="63.5" x2="116.84" y2="53.34" width="0.1524" layer="91"/>
-<wire x1="116.84" y1="53.34" x2="127" y2="53.34" width="0.1524" layer="91"/>
-<pinref part="C3" gate="G$1" pin="2"/>
-<junction x="116.84" y="53.34"/>
-<pinref part="D2" gate="1" pin="A"/>
-<wire x1="116.84" y1="63.5" x2="132.08" y2="63.5" width="0.1524" layer="91"/>
-<wire x1="116.84" y1="63.5" x2="116.84" y2="83.82" width="0.1524" layer="91"/>
-<junction x="116.84" y="63.5"/>
 <wire x1="-86.36" y1="-27.94" x2="-86.36" y2="83.82" width="0.1524" layer="91"/>
-<junction x="-86.36" y="83.82"/>
 <wire x1="-165.1" y1="144.78" x2="-165.1" y2="83.82" width="0.1524" layer="91"/>
 <junction x="-165.1" y="83.82"/>
@@
 <wire x1="83.82" y1="160.02" x2="83.82" y2="154.94" width="0.1524" layer="91"/>
 </segment>
-</net>
+<segment>
+<pinref part="U4" gate="G$1" pin="P$1"/>
+<pinref part="D2" gate="1" pin="A"/>
+<wire x1="116.84" y1="63.5" x2="132.08" y2="63.5" width="0.1524" layer="91"/>
+<wire x1="116.84" y1="63.5" x2="116.84" y2="53.34" width="0.1524" layer="91"/>
+<wire x1="116.84" y1="53.34" x2="127" y2="53.34" width="0.1524" layer="91"/>
+<pinref part="C3" gate="G$1" pin="2"/>
+<junction x="116.84" y="53.34"/>
+<label x="114.3" y="63.5" size="1.778" layer="95"/>
+</segment>
+</net>

Commit message: Changed mistakes...
Oh god
Connections:
- removed net N$69: R16.1, U10.P$4
- removed net N$75: R15.1, U11.P$4
- new net N$45: R16.1, U11.P$4
- new net N$9: R15.1, U10.P$4
Other:
- moved on the sheet: R16
Changed lines of the file:
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@@
 <?xml version="1.0" encoding="utf-8"?>
 <!DOCTYPE eagle SYSTEM "eagle.dtd">
-<eagle version="7.1.0">
+<eagle version="7.2.0">
 <drawing>
 <settings>
@@
 <instance part="R14" gate="G$1" x="-353.06" y="-60.96"/>
 <instance part="R15" gate="G$1" x="-414.02" y="-76.2"/>
-<instance part="R16" gate="G$1" x="-414.02" y="-91.44"/>
+<instance part="R16" gate="G$1" x="-350.52" y="-76.2"/>
 <instance part="U11" gate="G$1" x="-266.7" y="-63.5"/>
 <instance part="C21" gate="G$1" x="-284.48" y="-58.42" rot="R180"/>
@@
 </segment>
 </net>
-<net name="N$69" class="0">
-<segment>
-<pinref part="U10" gate="G$1" pin="P$4"/>
-<wire x1="-472.44" y1="-68.58" x2="-472.44" y2="-91.44" width="0.1524" layer="91"/>
-<pinref part="R16" gate="G$1" pin="1"/>
-<wire x1="-472.44" y1="-91.44" x2="-419.1" y2="-91.44" width="0.1524" layer="91"/>
-</segment>
-</net>
-<net name="N$70" class="0">
-<segment>
-<pinref part="R16" gate="G$1" pin="2"/>
-<wire x1="-408.94" y1="-91.44" x2="-342.9" y2="-91.44" width="0.1524" layer="91"/>
-<pinref part="Q13" gate="G$1" pin="G"/>
-<wire x1="-342.9" y1="-91.44" x2="-342.9" y2="-76.2" width="0.1524" layer="91"/>
-</segment>
-</net>
 <net name="N$71" class="0">
 <segment>
@@
 </segment>
 </net>
-<net name="N$75" class="0">
-<segment>
-<pinref part="U11" gate="G$1" pin="P$4"/>
-<wire x1="-274.32" y1="-71.12" x2="-274.32" y2="-101.6" width="0.1524" layer="91"/>
-<wire x1="-274.32" y1="-101.6" x2="-424.18" y2="-101.6" width="0.1524" layer="91"/>
-<wire x1="-424.18" y1="-101.6" x2="-424.18" y2="-76.2" width="0.1524" layer="91"/>
-<pinref part="R15" gate="G$1" pin="1"/>
-<wire x1="-424.18" y1="-76.2" x2="-419.1" y2="-76.2" width="0.1524" layer="91"/>
-</segment>
-</net>
 <net name="N$76" class="0">
 <segment>
@@
 </segment>
 </net>
+<net name="N$9" class="0">
+<segment>
+<pinref part="R15" gate="G$1" pin="1"/>
+<pinref part="U10" gate="G$1" pin="P$4"/>
+<wire x1="-472.44" y1="-68.58" x2="-472.44" y2="-76.2" width="0.1524" layer="91"/>
+<wire x1="-472.44" y1="-76.2" x2="-419.1" y2="-76.2" width="0.1524" layer="91"/>
+</segment>
+</net>
+<net name="N$45" class="0">
+<segment>
+<pinref part="U11" gate="G$1" pin="P$4"/>
+<wire x1="-274.32" y1="-71.12" x2="-274.32" y2="-93.98" width="0.1524" layer="91"/>
+<wire x1="-274.32" y1="-93.98" x2="-355.6" y2="-93.98" width="0.1524" layer="91"/>
+<pinref part="R16" gate="G$1" pin="1"/>
+<wire x1="-355.6" y1="-93.98" x2="-355.6" y2="-76.2" width="0.1524" layer="91"/>
+</segment>
+</net>
+<net name="N$46" class="0">
+<segment>
+<pinref part="R16" gate="G$1" pin="2"/>
+<pinref part="Q13" gate="G$1" pin="G"/>
+<wire x1="-345.44" y1="-76.2" x2="-342.9" y2="-76.2" width="0.1524" layer="91"/>
+</segment>
+</net>
