File: motordriver.sch (EAGLE design)
At the start: 98 parts, among them J1 CONNECTOR_MOTORS, J10 HEADER_1X3, J11 HEADER_1X3, J2 CONNECTOR_MOTORS, J3 CONNECTOR_MOTORS, J4 CONNECTOR_MOTORS, J5 HEADER_1X3, J6 HEADER_1X3, J7 HEADER_1X3, J8 HEADER_1X3, J9 CONNECTOR_MOTORS, Q1 MOSFET, Q10 MOSFET, Q11 MOSFET, Q12 MOSFET, Q13 MOSFET, Q14 MOSFET, Q15 MOSFET, Q16 MOSFET, Q2 MOSFET, Q3 MOSFET, Q4 MOSFET, Q5 MOSFET, Q6 MOSFET, Q7 MOSFET, Q8 MOSFET, Q9 MOSFET, U1 74XX139_PDIP, U10 IR2111_PDIP, U11 IR2111_PDIP, U12 7812_TO220, U2 TL084_PDIP, U3 7812_TO220, U4 IR2111_PDIP, U5 IR2111_PDIP, U6 IR2111_PDIP, U7 IR2111_PDIP, U8 IR2111_PDIP, U9 IR2111_PDIP

Commit message: Routing Adventure Part I
Its never ogre.
Connections:
- net GND renamed GND_32
- net VCC_12V: now also U$1.IN
- net V_IN: no longer U$1.IN
Changed lines of the file:
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@@
 <label x="-76.2" y="134.62" size="1.778" layer="95" rot="R90"/>
 </segment>
-</net>
-<net name="GND" class="0">
+<segment>
+<pinref part="U$1" gate="G$1" pin="IN"/>
+<wire x1="-360.68" y1="-78.74" x2="-365.76" y2="-78.74" width="0.1524" layer="91"/>
+<label x="-368.3" y="-78.74" size="1.778" layer="95"/>
+</segment>
+</net>
+<net name="GND_32" class="0">
 <segment>
 <pinref part="U3" gate="G$1" pin="GND"/>
@@
 <net name="V_IN" class="0">
 <segment>
-<pinref part="U$1" gate="G$1" pin="IN"/>
-<wire x1="-360.68" y1="-78.74" x2="-365.76" y2="-78.74" width="0.1524" layer="91"/>
-<label x="-368.3" y="-78.74" size="1.778" layer="95"/>
-</segment>
-<segment>
 <pinref part="U12" gate="G$1" pin="IN"/>

Commit message: TIS FUCKING DONE
Connections:
- removed net VIN_RAW: J9.+, U3.IN
- net V_IN: now also J9.+, U3.IN
Changed lines of the file:
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@@
 <label x="66.04" y="-5.08" size="1.778" layer="95"/>
+</segment>
+<segment>
+<label x="-208.28" y="116.84" size="1.778" layer="95"/>
+<pinref part="J9" gate="G$1" pin="+"/>
+<wire x1="-226.06" y1="116.84" x2="-203.2" y2="116.84" width="0.1524" layer="91"/>
+<wire x1="-203.2" y1="116.84" x2="-203.2" y2="93.98" width="0.1524" layer="91"/>
+<pinref part="U3" gate="G$1" pin="IN"/>
+<wire x1="-203.2" y1="93.98" x2="-193.04" y2="93.98" width="0.1524" layer="91"/>
 </segment>
 </net>
@@
 </segment>
 </net>
-<net name="VIN_RAW" class="0">
-<segment>
-<label x="-208.28" y="116.84" size="1.778" layer="95"/>
-<pinref part="J9" gate="G$1" pin="+"/>
-<wire x1="-226.06" y1="116.84" x2="-203.2" y2="116.84" width="0.1524" layer="91"/>
-<pinref part="U3" gate="G$1" pin="IN"/>
-<wire x1="-203.2" y1="93.98" x2="-193.04" y2="93.98" width="0.1524" layer="91"/>
-<label x="-200.66" y="93.98" size="1.778" layer="95"/>
-<wire x1="-203.2" y1="116.84" x2="-203.2" y2="93.98" width="0.1524" layer="91"/>
-</segment>
-</net>

Commit message: SHIP IT!
Connections:
- removed net N$6: R23.1
- net GND_32: now also R23.1
Changed lines of the file:
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@@
 </segment>
 <segment>
+<pinref part="R23" gate="G$1" pin="1"/>
 <pinref part="GND32" gate="1" pin="GND"/>
-<wire x1="-73.66" y1="106.68" x2="-73.66" y2="101.6" width="0.1524" layer="91"/>
+<wire x1="-73.66" y1="109.22" x2="-73.66" y2="101.6" width="0.1524" layer="91"/>
 </segment>
 </net>
@@
 <wire x1="33.02" y1="40.64" x2="35.56" y2="40.64" width="0.1524" layer="91"/>
 <wire x1="33.02" y1="43.18" x2="33.02" y2="40.64" width="0.1524" layer="91"/>
+<junction x="33.02" y="40.64"/>
 </segment>
 </net>
@@
 <wire x1="40.64" y1="40.64" x2="66.04" y2="40.64" width="0.1524" layer="91"/>
 <wire x1="40.64" y1="43.18" x2="40.64" y2="40.64" width="0.1524" layer="91"/>
+<junction x="40.64" y="40.64"/>
 </segment>
 </net>
@@
 <wire x1="33.02" y1="-30.48" x2="35.56" y2="-30.48" width="0.1524" layer="91"/>
 <wire x1="33.02" y1="-27.94" x2="33.02" y2="-30.48" width="0.1524" layer="91"/>
+<junction x="33.02" y="-30.48"/>
 </segment>
 </net>
@@
 <wire x1="40.64" y1="-30.48" x2="66.04" y2="-30.48" width="0.1524" layer="91"/>
 <wire x1="40.64" y1="-27.94" x2="40.64" y2="-30.48" width="0.1524" layer="91"/>
+<junction x="40.64" y="-30.48"/>
 </segment>
 </net>
@@
 <wire x1="-368.3" y1="45.72" x2="-365.76" y2="45.72" width="0.1524" layer="91"/>
 <wire x1="-368.3" y1="48.26" x2="-368.3" y2="45.72" width="0.1524" layer="91"/>
+<junction x="-368.3" y="45.72"/>
 </segment>
 </net>
@@
 <wire x1="-360.68" y1="45.72" x2="-335.28" y2="45.72" width="0.1524" layer="91"/>
 <wire x1="-360.68" y1="45.72" x2="-360.68" y2="48.26" width="0.1524" layer="91"/>
+<junction x="-360.68" y="45.72"/>
 </segment>
 </net>
@@
 <wire x1="-368.3" y1="-33.02" x2="-365.76" y2="-33.02" width="0.1524" layer="91"/>
 <wire x1="-368.3" y1="-30.48" x2="-368.3" y2="-33.02" width="0.1524" layer="91"/>
+<junction x="-368.3" y="-33.02"/>
 </segment>
 </net>
@@
 <wire x1="-360.68" y1="-33.02" x2="-335.28" y2="-33.02" width="0.1524" layer="91"/>
 <wire x1="-360.68" y1="-30.48" x2="-360.68" y2="-33.02" width="0.1524" layer="91"/>
+<junction x="-360.68" y="-33.02"/>
 </segment>
 </net>
@@
 </segment>
 </net>
-<net name="N$6" class="0">
-<segment>
-<pinref part="R23" gate="G$1" pin="1"/>
-<wire x1="-73.66" y1="109.22" x2="-73.66" y2="106.68" width="0.1524" layer="91"/>
-</segment>
-</net>

Commit message: Front side labels...COMPLETE
IT tAkes AlOT of COoKs to mAke A STew.
Parts:
- renumbered U$2 to ENC
Changed lines of the file:
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@@
 <part name="J7" library="motordriverslib" deviceset="HEADER_1X3" device=""/>
 <part name="J8" library="motordriverslib" deviceset="HEADER_1X3" device=""/>
-<part name="U$2" library="motordriverslib" deviceset="CONN_5X2" device=""/>
+<part name="ENC" library="motordriverslib" deviceset="CONN_5X2" device=""/>
 <part name="R17" library="motordriverslib" deviceset="RES_SMT" device=""/>
 <part name="R18" library="motordriverslib" deviceset="RES_SMT" device=""/>
@@
 <instance part="J7" gate="G$1" x="-213.36" y="10.16"/>
 <instance part="J8" gate="G$1" x="-144.78" y="5.08" rot="MR0"/>
-<instance part="U$2" gate="G$1" x="-111.76" y="-99.06"/>
+<instance part="ENC" gate="G$1" x="-111.76" y="-99.06"/>
 <instance part="R17" gate="G$1" x="-121.92" y="71.12" rot="R90"/>
 <instance part="R18" gate="G$1" x="-121.92" y="50.8" rot="R90"/>
@@
 </segment>
 <segment>
-<pinref part="U$2" gate="G$1" pin="P$10"/>
+<pinref part="ENC" gate="G$1" pin="P$10"/>
 <pinref part="GND28" gate="1" pin="GND"/>
 <wire x1="-116.84" y1="-73.66" x2="-137.16" y2="-73.66" width="0.1524" layer="91"/>
@@
 </segment>
 <segment>
-<pinref part="U$2" gate="G$1" pin="P$1"/>
+<pinref part="ENC" gate="G$1" pin="P$1"/>
 <pinref part="GND29" gate="1" pin="GND"/>
 <wire x1="-116.84" y1="-96.52" x2="-137.16" y2="-96.52" width="0.1524" layer="91"/>
@@
 </segment>
 <segment>
-<pinref part="U$2" gate="G$1" pin="P$2"/>
+<pinref part="ENC" gate="G$1" pin="P$2"/>
 <wire x1="-116.84" y1="-93.98" x2="-127" y2="-93.98" width="0.1524" layer="91"/>
 <label x="-129.54" y="-93.98" size="1.778" layer="95"/>
 </segment>
 <segment>
-<pinref part="U$2" gate="G$1" pin="P$9"/>
+<pinref part="ENC" gate="G$1" pin="P$9"/>
 <wire x1="-116.84" y1="-76.2" x2="-127" y2="-76.2" width="0.1524" layer="91"/>
 <label x="-129.54" y="-76.2" size="1.778" layer="95"/>
@@
 <net name="X_A" class="0">
 <segment>
-<pinref part="U$2" gate="G$1" pin="P$4"/>
+<pinref part="ENC" gate="G$1" pin="P$4"/>
 <wire x1="-116.84" y1="-88.9" x2="-127" y2="-88.9" width="0.1524" layer="91"/>
 <label x="-127" y="-88.9" size="1.778" layer="95"/>
@@
 <net name="Y_A" class="0">
 <segment>
-<pinref part="U$2" gate="G$1" pin="P$7"/>
+<pinref part="ENC" gate="G$1" pin="P$7"/>
 <wire x1="-127" y1="-81.28" x2="-116.84" y2="-81.28" width="0.1524" layer="91"/>
 <label x="-127" y="-81.28" size="1.778" layer="95"/>
@@
 <net name="Y_B" class="0">
 <segment>
-<pinref part="U$2" gate="G$1" pin="P$6"/>
+<pinref part="ENC" gate="G$1" pin="P$6"/>
 <wire x1="-116.84" y1="-83.82" x2="-127" y2="-83.82" width="0.1524" layer="91"/>
 <label x="-127" y="-83.82" size="1.778" layer="95"/>
@@
 <net name="X_B" class="0">
 <segment>
-<pinref part="U$2" gate="G$1" pin="P$5"/>
+<pinref part="ENC" gate="G$1" pin="P$5"/>
 <wire x1="-116.84" y1="-86.36" x2="-127" y2="-86.36" width="0.1524" layer="91"/>
 <label x="-127" y="-86.36" size="1.778" layer="95"/>
